Commit message: Update arm4.urdf

File: data/arm4.urdf (robot description, URDF)
Before this commit: robot arm4, 6 links, 5 joints
Joints:
- joint joint1_yaw: origin xyz=0 0 0.045 -> xyz=0 0 0.043
- joint joint2_shoulder: origin xyz=0 0 0.045 -> xyz=0 0 0.044
- joint joint3_elbow: origin xyz=0 0 0.115 -> xyz=0 0 0.110
- joint joint4_mount: origin xyz=0 0 0.105 -> xyz=0 0 0.133

Commit message: Update arm4.urdf

File: data/arm4.urdf (robot description, URDF)
Before this commit: robot arm4, 6 links, 5 joints
Joints:
- joint joint4_mount: origin xyz=0 0 0.133 -> xyz=0 0 0.100

Commit message: Update arm4.urdf

File: data/arm4.urdf (robot description, URDF)
Before this commit: robot arm4, 6 links, 5 joints
Links:
- removed link gripper_base
- link base_link: mass 0.05 -> 0.1; geometry visual mesh filename=base_link.stl scale=0.001 0.001 0.001
- link link1: geometry visual mesh filename=link1.stl scale=0.001 0.001 0.001
- link link2: geometry visual mesh filename=link2.stl scale=0.001 0.001 0.001
- link moving_jaw: mass 0.05 -> 0.02; geometry visual mesh filename=moving_jaw.stl scale=0.001 0.001 0.001
- link shoulder: geometry visual mesh filename=shoulder.stl scale=0.001 0.001 0.001
Joints:
- removed joint joint4_mount
- joint gripper_joint: axis 1 0 0 -> -1 0 0; origin xyz=-0.047 0 0.010 -> xyz=0 0 0; parent gripper_base -> link2
- joint joint1_yaw: origin xyz=0 0 0.043 -> xyz=0.00423 -0.00962 0
- joint joint2_shoulder: origin xyz=0 0 0.044 -> xyz=0 -0.00159 0.06446
- joint joint3_elbow: origin xyz=0 0 0.110 -> xyz=0 0.00590 0.10894

Commit message: Update arm4.urdf

File: data/arm4.urdf (robot description, URDF)
Before this commit: robot arm4, 5 links, 4 joints
Joints:
- joint gripper_joint: axis -1 0 0 -> 0 1 0
- joint joint2_shoulder: axis 1 0 0 -> 0 1 0
- joint joint3_elbow: axis 1 0 0 -> 0 1 0

Commit message: Update arm4.urdf

File: data/arm4.urdf (robot description, URDF)
Before this commit: robot arm4, 5 links, 4 joints
Joints:
- joint joint2_shoulder: axis 0 1 0 -> 0 -1 0
- joint joint3_elbow: axis 0 1 0 -> 0 -1 0

Commit message: Update arm4.urdf

File: data/arm4.urdf (robot description, URDF)
Before this commit: robot arm4, 5 links, 4 joints
Joints:
- joint gripper_joint: limit lower=0 upper=0.030 effort=5 velocity=0.1 -> lower=-0.0208 upper=0.0092 effort=5 velocity=0.1

Commit message: Update arm4.urdf

File: data/arm4.urdf (robot description, URDF)
Before this commit: robot arm4, 5 links, 4 joints
Joints:
- joint joint2_shoulder: origin xyz=0 -0.00159 0.06446 -> xyz=0 -0.00159 0.07446
